Commit message: fix(jointstate): reverse _ to space

File: src/komarm/urdf/komarm.urdf (robot description, URDF)
Before this commit: robot arm_main, 6 links, 5 joints
Joints:
- removed joint Revolute_11
- removed joint Revolute_12
- removed joint Revolute_7
- removed joint Revolute_8
- removed joint Revolute_9
- added joint Revolute 11: type revolute, parent base_mount_v2_1, child servo_holder_v23_3, origin xyz=0.02255 -0.0369 0.029 rpy=0 0 0, axis -1.0 -0.0 -0.0, limit lower=-3.141593 upper=0.0 effort=100 velocity=100
- added joint Revolute 12: type revolute, parent base_link, child base_mount_v2_1, origin xyz=-0.00135 0.0369 -0.0165 rpy=0 0 0, axis 0.0 -0.0 -1.0, limit lower=-1.570796 upper=1.570796 effort=100 velocity=100
- added joint Revolute 7: type revolute, parent servo_holder_v23_3, child servo_holder2_v9_1, origin xyz=0.0005 0.0324 0.02945 rpy=0 0 0, axis 1.0 -0.0 0.0, limit lower=-3.141593 upper=0.0 effort=100 velocity=100
- added joint Revolute 8: type revolute, parent servo_holder2_v9_1, child hand_rotation_v13_4, origin xyz=0.001 -0.0662 0.0 rpy=0 0 0, axis 1.0 0.0 0.0, limit lower=-0.349066 upper=1.570796 effort=100 velocity=100
- added joint Revolute 9: type continuous, parent hand_rotation_v13_4, child hand_v17_1, origin xyz=-0.0232 -0.0554 0.0 rpy=0 0 0, axis -0.0 1.0 0.0

Commit message: feat(urdf): change to package path

File: src/komarm/urdf/komarm.urdf (robot description, URDF)
Before this commit: robot arm_main, 6 links, 5 joints
Links:
- link base_link: geometry collision mesh filename=package://komarm/meshes/base_link.stl scale=0.001 0.001 0.001; visual mesh filename=package://komarm/meshes/base_link.stl scale=0.001 0.001 0.001
- link base_mount_v2_1: geometry collision mesh filename=package://komarm/meshes/base_mount_v2_1.stl scale=0.001 0.001 0.001; visual mesh filename=package://komarm/meshes/base_mount_v2_1.stl scale=0.001 0.001 0.001
- link hand_rotation_v13_4: geometry collision mesh filename=package://komarm/meshes/hand_rotation_v13_4.stl scale=0.001 0.001 0.001; visual mesh filename=package://komarm/meshes/hand_rotation_v13_4.stl scale=0.001 0.001 0.001
- link hand_v17_1: geometry collision mesh filename=package://komarm/meshes/hand_v17_1.stl scale=0.001 0.001 0.001; visual mesh filename=package://komarm/meshes/hand_v17_1.stl scale=0.001 0.001 0.001
- link servo_holder2_v9_1: geometry collision mesh filename=package://komarm/meshes/servo_holder2_v9_1.stl scale=0.001 0.001 0.001; visual mesh filename=package://komarm/meshes/servo_holder2_v9_1.stl scale=0.001 0.001 0.001
- link servo_holder_v23_3: geometry collision mesh filename=package://komarm/meshes/servo_holder_v23_3.stl scale=0.001 0.001 0.001; visual mesh filename=package://komarm/meshes/servo_holder_v23_3.stl scale=0.001 0.001 0.001

Commit message: fix(urdf): revert

File: src/komarm/urdf/komarm.urdf (robot description, URDF)
Before this commit: robot arm_main, 6 links, 5 joints
Links:
- link base_link: geometry collision mesh filename=../meshes/base_link.stl scale=0.001 0.001 0.001; visual mesh filename=../meshes/base_link.stl scale=0.001 0.001 0.001
- link base_mount_v2_1: geometry collision mesh filename=../meshes/base_mount_v2_1.stl scale=0.001 0.001 0.001; visual mesh filename=../meshes/base_mount_v2_1.stl scale=0.001 0.001 0.001
- link hand_rotation_v13_4: geometry collision mesh filename=../meshes/hand_rotation_v13_4.stl scale=0.001 0.001 0.001; visual mesh filename=../meshes/hand_rotation_v13_4.stl scale=0.001 0.001 0.001
- link hand_v17_1: geometry collision mesh filename=../meshes/hand_v17_1.stl scale=0.001 0.001 0.001; visual mesh filename=../meshes/hand_v17_1.stl scale=0.001 0.001 0.001
- link servo_holder2_v9_1: geometry collision mesh filename=../meshes/servo_holder2_v9_1.stl scale=0.001 0.001 0.001; visual mesh filename=../meshes/servo_holder2_v9_1.stl scale=0.001 0.001 0.001
- link servo_holder_v23_3: geometry collision mesh filename=../meshes/servo_holder_v23_3.stl scale=0.001 0.001 0.001; visual mesh filename=../meshes/servo_holder_v23_3.stl scale=0.001 0.001 0.001
